Commit message: modify gazebo

File: treebo_description/urdf/robot.urdf.xacro (robot description, xacro)
@@ -2,3 +2,6 @@
 <robot name="treebo" xmlns:xacro="http://www.ros.org/wiki/xacro">
     <xacro:include filename="robot_core.xacro"/>
+    <xacro:include filename="lidar.xacro" />
+    <xacro:include filename="robot_gazebo.xacro"/>
+    <xacro:include filename="gazebo_control.xacro"/>
 </robot>

File: treebo_description/urdf/robot_core.xacro (robot description, xacro)
@@ -105,3 +105,64 @@
         <axis xyz="0 0 -1"/>
     </joint>
+    <link name="lidar_mount">
+        <visual>
+            <origin xyz="0 0 0" rpy="0 0 0"/>
+            <geometry>
+                <cylinder radius="0.025" length="0.02"/>
+            </geometry>
+            <material name="black">
+                <color rgba="0 0 0 1"/>
+            </material>
+        </visual>
+        <collision>
+            <origin xyz="0 0 0" rpy="0 0 0"/>
+            <geometry>
+                <cylinder radius="0.025" length="0.02"/>
+            </geometry>
+        </collision>
+        <inertial>
+            <origin xyz="0 0 0" rpy="0 0 0"/>
+            <mass value="0.05"/>
+            <!-- 대략적인 관성치 m*r^2/2, m*(3r^2+h^2)/12 등 근사 -->
+            <inertia ixx="3.0e-05" ixy="0" ixz="0" iyy="3.0e-05" iyz="0" izz="3.0e-05"/>
+        </inertial>
+    </link>
+    <!-- 마운트를 섀시에 고정 -->
+    <joint name="lidar_mount_fixed_joint" type="fixed">
+        <parent link="chassis"/>
+        <child link="lidar_mount"/>
+        <!-- 섀시 위쪽 중앙에 배치. 필요시 xyz 조정 -->
+        <origin xyz="0.0 0.0 0.09" rpy="0 0 0"/>
+    </joint>
+    <!-- 레이저 링크 라이다 본체를 단순 실린더로 표현 -->
+    <link name="laser_link">
+        <visual>
+            <origin xyz="0 0 0" rpy="0 0 0"/>
+            <geometry>
+            <!-- 지름 약 6cm, 높이 6cm 정도의 라이다로 가정 -->
+                <cylinder radius="0.03" length="0.06"/>
+            </geometry>
+            <material name="blue">
+                <color rgba="0.2 0.2 1 1"/>
+            </material>
+        </visual>
+        <collision>
+            <origin xyz="0 0 0" rpy="0 0 0"/>
+            <geometry>
+                <cylinder radius="0.03" length="0.06"/>
+            </geometry>
+        </collision>
+        <inertial>
+            <origin xyz="0 0 0" rpy="0 0 0"/>
+            <mass value="0.2"/>
+            <inertia ixx="1.2e-04" ixy="0" ixz="0" iyy="1.2e-04" iyz="0" izz="1.6e-04"/>
+        </inertial>
+    </link>
+    <!-- 레이저를 마운트 위에 고정 -->
+    <joint name="laser_link_fixed_joint" type="fixed">
+    <parent link="lidar_mount"/>
+    <child link="laser_link"/>
+    <!-- 살짝 위로 올리고 뒤집어서 전방 스캔면 정렬 -->
+    <origin xyz="0.0 0.0 0.05" rpy="0 0 ${pi}"/>
+    </joint>
 </robot>
