Commit message: Add sllidar_ros2 as submodule

File: treebo_description/urdf/robot_core.xacro (robot description, xacro)
@@ -163,6 +163,5 @@
     <parent link="lidar_mount"/>
     <child link="laser_link"/>
-    <!-- 살짝 위로 올리고 뒤집어서 전방 스캔면 정렬 -->
-    <origin xyz="0.0 0.0 0.05" rpy="0 0 ${pi}"/>
+    <origin xyz="0.0 0.0 0.05" rpy="0 0 0"/>
     </joint>
 </robot>

Commit message: update

File: treebo_description/urdf/robot_core.xacro (robot description, xacro)
@@ -44,6 +44,7 @@
     <joint name="front_left_wheel_joint" type="continuous">
         <parent link="base_link"/>
-        <child link="front_left_wheel"/>
-        <origin xyz="0.12 0.175 0" rpy="-${pi/2} 0 0"/>
+        <child  link="front_left_wheel"/>
+        <!-- x = +0.095, y = +0.1075 -->
+        <origin xyz="0.095 0.1075 0" rpy="-${pi/2} 0 0"/>
         <axis xyz="0 0 1"/>
     </joint>
@@ -63,6 +64,7 @@
     <joint name="front_right_wheel_joint" type="continuous">
         <parent link="base_link"/>
-        <child link="front_right_wheel"/>
-        <origin xyz="0.12 -0.175 0" rpy="${pi/2} 0 0"/>
+        <child  link="front_right_wheel"/>
+        <!-- x = +0.095, y = -0.1075 -->
+        <origin xyz="0.095 -0.1075 0" rpy="${pi/2} 0 0"/>
         <axis xyz="0 0 -1"/>
     </joint>
@@ -82,6 +84,7 @@
     <joint name="rear_left_wheel_joint" type="continuous">
         <parent link="base_link"/>
-        <child link="rear_left_wheel"/>
-        <origin xyz="-0.12 0.175 0" rpy="-${pi/2} 0 0"/>
+        <child  link="rear_left_wheel"/>
+        <!-- x = -0.095, y = +0.1075 -->
+        <origin xyz="-0.095 0.1075 0" rpy="-${pi/2} 0 0"/>
         <axis xyz="0 0 1"/>
     </joint>
@@ -101,6 +104,7 @@
     <joint name="rear_right_wheel_joint" type="continuous">
         <parent link="base_link"/>
-        <child link="rear_right_wheel"/>
-        <origin xyz="-0.12 -0.175 0" rpy="${pi/2} 0 0"/>
+        <child  link="rear_right_wheel"/>
+        <!-- x = -0.095, y = -0.1075 -->
+        <origin xyz="-0.095 -0.1075 0" rpy="${pi/2} 0 0"/>
         <axis xyz="0 0 -1"/>
     </joint>
