Commit message: treebo_car_version

File: treebo_description/urdf/gazebo_control.xacro (robot description, xacro)
@@ -9,6 +9,6 @@
         <right_joint>rear_right_wheel_joint</right_joint>
         <!-- 실제 치수 -->
-        <wheel_separation>0.35</wheel_separation>
-        <wheel_radius>0.05</wheel_radius>
+        <wheel_separation>0.20</wheel_separation>
+        <wheel_radius>0.04</wheel_radius>
         <!-- ROS <-> GZ 브리지 토픽 -->
         <topic>cmd_vel</topic>

File: treebo_description/urdf/robot_core.xacro (robot description, xacro)
@@ -12,14 +12,14 @@
     <link name="chassis">
         <visual>
-            <origin xyz="0.1 0 0.075"/>
+            <origin xyz="0 0 0.075"/>
             <geometry><box size="0.4 0.3 0.1"/></geometry>
             <material name="white"/>
         </visual>
         <collision>
-            <origin xyz="0.1 0 0.075"/>
+            <origin xyz="0 0 0.075"/>
             <geometry><box size="0.4 0.3 0.1"/></geometry>
         </collision>
         <xacro:inertial_box mass="0.4" x="0.4" y="0.3" z="0.1">
-        <origin xyz="0.1 0 0.075" rpy="0 0 0"/>
+        <origin xyz="0 0 0.075" rpy="0 0 0"/>
         </xacro:inertial_box>
     </link>
@@ -27,5 +27,5 @@
         <parent link="base_link"/>
         <child link="chassis"/>
-        <origin xyz="-0.1 0 0"/>
+        <origin xyz="0 0 0"/>
     </joint>
     <!-- FRONT LEFT -->
@@ -137,5 +137,5 @@
         <child link="lidar_mount"/>
         <!-- 섀시 위쪽 중앙에 배치. 필요시 xyz 조정 -->
-        <origin xyz="0.0 0.0 0.09" rpy="0 0 0"/>
+        <origin xyz="-0.085 0.0 0.09" rpy="0 0 0"/>
     </joint>
     <!-- 레이저 링크 라이다 본체를 단순 실린더로 표현 -->

Commit message: slam&nav

File: treebo_description/urdf/gazebo_control.xacro (robot description, xacro)
@@ -9,6 +9,6 @@
         <right_joint>rear_right_wheel_joint</right_joint>
         <!-- 실제 치수 -->
-        <wheel_separation>0.20</wheel_separation>
-        <wheel_radius>0.04</wheel_radius>
+        <wheel_separation>0.50</wheel_separation>
+        <wheel_radius>0.05</wheel_radius>
         <!-- ROS <-> GZ 브리지 토픽 -->
         <topic>cmd_vel</topic>

File: treebo_description/urdf/robot_core.xacro (robot description, xacro)
@@ -13,12 +13,12 @@
         <visual>
             <origin xyz="0 0 0.075"/>
-            <geometry><box size="0.4 0.3 0.1"/></geometry>
+            <geometry><box size="0.30 0.50 0.10"/></geometry>
             <material name="white"/>
         </visual>
         <collision>
             <origin xyz="0 0 0.075"/>
-            <geometry><box size="0.4 0.3 0.1"/></geometry>
+            <geometry><box size="0.30 0.50 0.10"/></geometry>
         </collision>
-        <xacro:inertial_box mass="0.4" x="0.4" y="0.3" z="0.1">
+        <xacro:inertial_box mass="0.4" x="0.30" y="0.50" z="0.10">
         <origin xyz="0 0 0.075" rpy="0 0 0"/>
         </xacro:inertial_box>
@@ -46,5 +46,5 @@
         <child  link="front_left_wheel"/>
         <!-- x = +0.095, y = +0.1075 -->
-        <origin xyz="0.095 0.1075 0" rpy="-${pi/2} 0 0"/>
+        <origin xyz="0.10 0.25 0" rpy="-${pi/2} 0 0"/>
         <axis xyz="0 0 1"/>
     </joint>
@@ -66,5 +66,5 @@
         <child  link="front_right_wheel"/>
         <!-- x = +0.095, y = -0.1075 -->
-        <origin xyz="0.095 -0.1075 0" rpy="${pi/2} 0 0"/>
+        <origin xyz="0.10 -0.25 0" rpy="${pi/2} 0 0"/>
         <axis xyz="0 0 -1"/>
     </joint>
@@ -86,5 +86,5 @@
         <child  link="rear_left_wheel"/>
         <!-- x = -0.095, y = +0.1075 -->
-        <origin xyz="-0.095 0.1075 0" rpy="-${pi/2} 0 0"/>
+        <origin xyz="-0.10 0.25 0" rpy="-${pi/2} 0 0"/>
         <axis xyz="0 0 1"/>
     </joint>
@@ -106,5 +106,5 @@
         <child  link="rear_right_wheel"/>
         <!-- x = -0.095, y = -0.1075 -->
-        <origin xyz="-0.095 -0.1075 0" rpy="${pi/2} 0 0"/>
+        <origin xyz="-0.10 -0.25 0" rpy="${pi/2} 0 0"/>
         <axis xyz="0 0 -1"/>
     </joint>
@@ -137,5 +137,5 @@
         <child link="lidar_mount"/>
         <!-- 섀시 위쪽 중앙에 배치. 필요시 xyz 조정 -->
-        <origin xyz="-0.085 0.0 0.09" rpy="0 0 0"/>
+        <origin xyz="0.1 0.0 0.125" rpy="0 0 0"/>
     </joint>
     <!-- 레이저 링크 라이다 본체를 단순 실린더로 표현 -->
